File: transpose/transpose.sch (KiCad schematic (older format))
At the start: 5 parts

Commit message: updated schematic
Parts:
- added R? (x11): 10K, symbol R
Connections:
- wire segments 58 -> 82
Other:
- moved on the sheet: J?, U?
